Commit message: Add parsing of initial_state for position state interface

File: cartesian_controller_simulation/urdf/joint.urdf.xacro (robot description, xacro)
@@ -1,21 +1,23 @@
 <?xml version="1.0"?>
 <robot xmlns:xacro="http://www.ros.org/wiki/xacro">
-        <!-- Individual joint. -->
-        <xacro:macro name="joint_interface" params="name p d">
-                <joint name="${name}">
-                        <command_interface name="position">
-                                <param name="min">-1</param>
-                                <param name="max">1</param>
-                        </command_interface>
-                        <command_interface name="velocity">
-                                <param name="min">-1</param>
-                                <param name="max">1</param>
-                        </command_interface>
-                        <param name="p">${p}</param>
-                        <param name="d">${d}</param>
-                        <state_interface name="position"/>
-                        <state_interface name="velocity"/>
-                        <state_interface name="effort"/>
-                </joint>
-        </xacro:macro>
+  <!-- Individual joint. -->
+  <xacro:macro name="joint_interface" params="name p d init_val:=0">
+    <joint name="${name}">
+      <command_interface name="position">
+        <param name="min">-1</param>
+        <param name="max">1</param>
+      </command_interface>
+      <command_interface name="velocity">
+        <param name="min">-1</param>
+        <param name="max">1</param>
+      </command_interface>
+      <param name="p">${p}</param>
+      <param name="d">${d}</param>
+      <state_interface name="position">
+        <param name="initial_value">${init_val}</param>
+      </state_interface>
+      <state_interface name="velocity"/>
+      <state_interface name="effort"/>
+    </joint>
+  </xacro:macro>
 </robot>

File: cartesian_controller_simulation/urdf/robot.urdf.xacro (robot description, xacro)
@@ -1,311 +1,311 @@
 <?xml version="1.0"?>
 <robot name="robot" xmlns:xacro="http://ros.org/wiki/xacro">
-        <!--
+  <!--
         A fictitious robot model for testing purposes.
         The kinematics is roughly inspired by the universal robots ur10.
         -->
-        <xacro:include filename="$(find cartesian_controller_simulation)/urdf/joint.urdf.xacro"/>
-        <!-- ROS2 control interfaces -->
-        <ros2_control name="cartesian_controller_simulation" type="system">
-                <xacro:joint_interface name="joint1" p="1000" d="0.5" />
-                <xacro:joint_interface name="joint2" p="1000" d="0.5" />
-                <xacro:joint_interface name="joint3" p="500" d="0.5" />
-                <xacro:joint_interface name="joint4" p="100" d="0.5" />
-                <xacro:joint_interface name="joint5" p="10" d="0.5" />
-                <xacro:joint_interface name="joint6" p="10" d="0.5" />
-                <hardware>
-                        <plugin>cartesian_controller_simulation/Simulator</plugin>
-                        <param name="mujoco_model">$(arg mujoco_model)</param>
-                </hardware>
-        </ros2_control>
-        <!-- joint properties -->
-        <xacro:property name="joint_radius" value="0.02" />
-        <xacro:property name="joint_length" value="0.03" />
-        <!-- link properties -->
-        <xacro:property name="link_radius" value="0.01" />
-        <xacro:property name="link1_length" value="0.15" />
-        <xacro:property name="link2_length" value="0.5" />
-        <xacro:property name="link3_length" value="0.5" />
-        <xacro:property name="link4_length" value="0.15" />
-        <xacro:property name="link5_length" value="0.10" />
-        <xacro:property name="link6_length" value="0.05" />
-        <!-- colors -->
-        <material name="joint_part1">
-                <color rgba="0.525 0.713 0.662 1.0"/>
-        </material>
-        <material name="joint_part2">
-                <color rgba="0.462 0.196 0.411 1.0"/>
-        </material>
-        <material name="base">
-                <color rgba="0.956863 0.796078 0.631373 1.0"/>
-        </material>
-        <material name="tip">
-                <color rgba="0.956 0.450 0.243 1.0"/>
-        </material>
-        <material name="link1">
-                <color rgba="0.949 0.631 0.823 1.0"/>
-        </material>
-        <material name="link2">
-                <color rgba="0.133 0.827 0.435 1.0"/>
-        </material>
-        <material name="link3">
-                <color rgba="0.968 0.721 0.313 1.0"/>
-        </material>
-        <material name="link4">
-                <color rgba="0.52549 0.529412 0.647059 1.0"/>
-        </material>
-        <material name="link5">
-                <color rgba="0.478431 0.415686 0.662745 1.0"/>
-        </material>
-        <material name="link6">
-                <color rgba="0.988 0.580 0.450 1.0"/>
-        </material>
-        <!-- Connect to world -->
-        <link name="world" />
-        <joint name="world_joint" type="fixed">
-                <parent link="world" />
-                <child link = "base_link" />
-                <origin xyz="0.0 0.0 0.0" rpy="0.0 0.0 0.0" />
-        </joint>
-        <link name="base_link" >
-                <inertial>
-                        <origin xyz="0 0 ${joint_length / 2.0}" rpy="0 0 0"/>
-                        <mass value="1"/>
-                        <inertia ixx="1.0"  ixy="0"  ixz="0" iyy="1.0" iyz="0" izz="1.0" />
-                </inertial>
-                <visual name="base">
-                        <origin xyz="0 0 ${joint_length / 2.0}" rpy="0 0 0" />
-                        <geometry>
-                                <cylinder length="${joint_length}" radius="${joint_radius}"/>
-                        </geometry>
-                        <material name="base"/>
-                </visual>
-        </link>
-        <joint name="joint1" type="revolute">
-                <parent link="base_link" />
-                <child link = "link1" />
-                <origin xyz="0.0 0.0 ${3.0 / 2.0 * joint_length}" rpy="0.0 0.0 0.0" />
-                <axis xyz="0 0 1" />
-                <limit lower="${-2.0 * pi}" upper="${2.0 * pi}" effort="1.0" velocity="10.0"/>
-        </joint>
-        <link name="link1">
-                <inertial>
-                        <origin xyz="0 0 ${link1_length / 2.0}" rpy="0 0 0"/>
-                        <mass value="1"/>
-                        <inertia ixx="1.0"  ixy="0"  ixz="0" iyy="1.0" iyz="0" izz="1.0" />
-                </inertial>
-                <visual name="joint1">
-                        <origin xyz="0 0 0" rpy="0 0 0" />
-                        <geometry>
-                                <cylinder length="${joint_length}" radius="${joint_radius}"/>
-                        </geometry>
-                        <material name="link1"/>
-                </visual>
-                <visual name="link">
-                        <origin xyz="0 0 ${link1_length / 2.0}" rpy="0 0 0" />
-                        <geometry>
-                                <cylinder length="${link1_length}" radius="${link_radius}"/>
-                        </geometry>
-                </visual>
-                <visual name="joint2">
-                        <origin xyz="0 0 ${link1_length}" rpy="${pi / 2.0} 0 0" />
-                        <geometry>
-                                <cylinder length="${joint_length}" radius="${joint_radius}"/>
-                        </geometry>
-                </visual>
-        </link>
-        <joint name="joint2" type="revolute">
-                <parent link="link1" />
-                <child link = "link2" />
-                <origin xyz="0.0 ${joint_length} ${link1_length}" rpy="0.0 ${pi / 2.0} 0.0" />
-                <axis xyz="0 1 0" />
-                <limit lower="${-2.0 * pi}" upper="${2.0 * pi}" effort="1.0" velocity="10.0"/>
-        </joint>
-        <link name="link2">
-                <inertial>
-                        <origin xyz="0 0 ${link2_length / 2.0}" rpy="0 0 0"/>
-                        <mass value="1"/>
-                        <inertia ixx="1.0"  ixy="0"  ixz="0" iyy="1.0" iyz="0" izz="1.0" />
-                </inertial>
-                <visual name="joint2">
-                        <origin xyz="0 0 0" rpy="${pi / 2.0} 0 0" />
-                        <geometry>
-                                <cylinder length="${joint_length}" radius="${joint_radius}"/>
-                        </geometry>
-                        <material name="link2"/>
-                </visual>
-                <visual name="link">
-                        <origin xyz="0 0 ${link2_length / 2.0}" rpy="0 0 0" />
-                        <geometry>
-                                <cylinder length="${link2_length}" radius="${link_radius}"/>
-                        </geometry>
-                </visual>
-                <visual name="joint3">
-                        <origin xyz="0 0 ${link2_length}" rpy="${pi / 2.0} 0 0" />
-                        <geometry>
-                                <cylinder length="${joint_length}" radius="${joint_radius}"/>
-                        </geometry>
-                </visual>
-        </link>
-        <joint name="joint3" type="revolute">
-                <parent link="link2" />
-                <child link = "link3" />
-                <origin xyz="0.0 -${joint_length} ${link2_length}" rpy="0.0 0.0 0.0" />
-                <axis xyz="0 1 0" />
-                <limit lower="${-pi}" upper="${pi}" effort="1.0" velocity="10.0"/>
-        </joint>
-        <link name="link3">
-                <inertial>
-                        <origin xyz="0 0 ${link3_length / 2.0}" rpy="0 0 0"/>
-                        <mass value="1"/>
-                        <inertia ixx="1.0"  ixy="0"  ixz="0" iyy="1.0" iyz="0" izz="1.0" />
-                </inertial>
-                <visual name="joint3">
-                        <origin xyz="0 0 0" rpy="${pi / 2.0} 0 0" />
-                        <geometry>
-                                <cylinder length="${joint_length}" radius="${joint_radius}"/>
-                        </geometry>
-                        <material name="link3"/>
-                </visual>
-                <visual name="link">
-                        <origin xyz="0 0 ${link3_length / 2.0}" rpy="0 0 0" />
-                        <geometry>
-                                <cylinder length="${link3_length}" radius="${link_radius}"/>
-                        </geometry>
-                </visual>
-                <visual name="joint4">
-                        <origin xyz="0 0 ${link3_length}" rpy="${pi / 2.0} 0 0" />
-                        <geometry>
-                                <cylinder length="${joint_length}" radius="${joint_radius}"/>
-                        </geometry>
-                </visual>
-        </link>
-        <joint name="joint4" type="revolute">
-                <parent link="link3" />
-                <child link = "link4" />
-                <origin xyz="0.0 ${joint_length} ${link3_length}" rpy="0.0 ${pi / 2.0} 0.0" />
-                <axis xyz="0 1 0" />
-                <limit lower="${-2.0 * pi}" upper="${2.0 * pi}" effort="1.0" velocity="10.0"/>
-        </joint>
-        <link name="link4">
-                <inertial>
-                        <origin xyz="0 0 ${link4_length / 2.0}" rpy="0 0 0"/>
-                        <mass value="1"/>
-                        <inertia ixx="1.0"  ixy="0"  ixz="0" iyy="1.0" iyz="0" izz="1.0" />
-                </inertial>
-                <visual name="joint4">
-                        <origin xyz="0 0 0" rpy="${pi / 2.0} 0 0" />
-                        <geometry>
-                                <cylinder length="${joint_length}" radius="${joint_radius}"/>
-                        </geometry>
-                        <material name="link4"/>
-                </visual>
-                <visual name="link">
-                        <origin xyz="0 ${link4_length / 2.0} 0" rpy="${pi / 2.0} 0 0" />
-                        <geometry>
-                                <cylinder length="${link4_length}" radius="${link_radius}"/>
-                        </geometry>
-                </visual>
-                <visual name="joint5">
-                        <origin xyz="0 ${link4_length} 0" rpy="0 0 0" />
-                        <geometry>
-                                <cylinder length="${joint_length}" radius="${joint_radius}"/>
-                        </geometry>
-                </visual>
-        </link>
-        <joint name="joint5" type="revolute">
-                <parent link="link4" />
-                <child link = "link5" />
-                <origin xyz="0.0 ${link4_length} ${joint_length}" rpy="0.0 0.0 0.0" />
-                <axis xyz="0 0 1" />
-                <limit lower="${-2.0 * pi}" upper="${2.0 * pi}" effort="1.0" velocity="10.0"/>
-        </joint>
-        <link name="link5">
-                <inertial>
-                        <origin xyz="0 0 ${link5_length / 2.0}" rpy="0 0 0"/>
-                        <mass value="1"/>
-                        <inertia ixx="1.0"  ixy="0"  ixz="0" iyy="1.0" iyz="0" izz="1.0" />
-                </inertial>
-                <visual name="joint5">
-                        <origin xyz="0 0 0" rpy="0 0 0" />
-                        <geometry>
-                                <cylinder length="${joint_length}" radius="${joint_radius}"/>
-                        </geometry>
-                        <material name="link5"/>
-                </visual>
-                <visual name="link">
-                        <origin xyz="0 0 ${link5_length / 2.0}" rpy="0 0 0" />
-                        <geometry>
-                                <cylinder length="${link5_length}" radius="${link_radius}"/>
-                        </geometry>
-                </visual>
-                <visual name="joint6">
-                        <origin xyz="0 0 ${link5_length}" rpy="${pi / 2.0} 0 0" />
-                        <geometry>
-                                <cylinder length="${joint_length}" radius="${joint_radius}"/>
-                        </geometry>
-                </visual>
-        </link>
-        <joint name="joint6" type="revolute">
-                <parent link="link5" />
-                <child link = "link6" />
-                <origin xyz="0.0 ${joint_length} ${link5_length}" rpy="0.0 0.0 0.0" />
-                <axis xyz="0 1 0" />
-                <limit lower="${-2.0 * pi}" upper="${2.0 * pi}" effort="1.0" velocity="10.0"/>
-        </joint>
-        <link name="link6">
-                <inertial>
-                        <origin xyz="0 0 ${link6_length / 2.0}" rpy="0 0 0"/>
-                        <mass value="1"/>
-                        <inertia ixx="1.0"  ixy="0"  ixz="0" iyy="1.0" iyz="0" izz="1.0" />
-                </inertial>
-                <visual name="joint6">
-                        <origin xyz="0 0 0" rpy="${pi / 2.0} 0 0" />
-                        <geometry>
-                                <cylinder length="${joint_length}" radius="${joint_radius}"/>
-                        </geometry>
-                        <material name="link6"/>
-                </visual>
-                <visual name="link">
-                        <origin xyz="0 ${link6_length / 2.0} 0" rpy="${-pi / 2.0} 0 0" />
-                        <geometry>
-                                <cylinder length="${link6_length}" radius="${link_radius}"/>
-                        </geometry>
-                </visual>
-        </link>
-        <!-- Attach a sensor link -->
-        <joint name="sensor_link_joint" type="fixed">
-                <origin xyz="0 ${link6_length / 2.0} 0" rpy="${-pi / 2.0} 0 0"/>
-                <parent link="link6"/>
-                <child link="sensor_link"/>
-        </joint>
-        <link name="sensor_link"/>
-        <!-- The default end-effector -->
-        <joint name="tool0_joint" type="fixed">
-                <origin xyz="0 0 ${link6_length / 2.0}" rpy="0 0 0"/>
-                <parent link="sensor_link"/>
-                <child link="tool0"/>
-        </joint>
-        <link name="tool0">
-                <visual>
-                        <origin xyz="0 0 0" rpy="0 0 0" />
-                        <geometry>
-                                <sphere radius="${link_radius}"/>
-                        </geometry>
-                        <material name="tip"/>
-                </visual>
-        </link>
-        <!-- Additional links for integration tests. -->
-        <joint name="invalid_sensor_link_joint" type="fixed">
-                <origin xyz="0 ${link6_length / 2.0} 0" rpy="${-pi / 2.0} 0 0"/>
-                <parent link="link6"/>
-                <child link="invalid_sensor_link"/>
-        </joint>
-        <link name="invalid_sensor_link"/>
-        <joint name="invalid_compliance_link_joint" type="fixed">
-                <origin xyz="0 0 0" rpy="0 0 0"/>
-                <parent link="sensor_link"/>
-                <child link="invalid_compliance_link"/>
-        </joint>
-        <link name="invalid_compliance_link"/>
+  <xacro:include filename="$(find cartesian_controller_simulation)/urdf/joint.urdf.xacro"/>
+  <!-- ROS2 control interfaces -->
+  <ros2_control name="cartesian_controller_simulation" type="system">
+    <xacro:joint_interface name="joint1" p="1000" d="0.5"/>
+    <xacro:joint_interface name="joint2" p="1000" d="0.5" init_val="-0.5"/>
+    <xacro:joint_interface name="joint3" p="500" d="0.5"/>
+    <xacro:joint_interface name="joint4" p="100" d="0.5"/>
+    <xacro:joint_interface name="joint5" p="10" d="0.5"/>
+    <xacro:joint_interface name="joint6" p="10" d="0.5"/>
+    <hardware>
+      <plugin>cartesian_controller_simulation/Simulator</plugin>
+      <param name="mujoco_model">$(arg mujoco_model)</param>
+    </hardware>
+  </ros2_control>
+  <!-- joint properties -->
+  <xacro:property name="joint_radius" value="0.02"/>
+  <xacro:property name="joint_length" value="0.03"/>
+  <!-- link properties -->
+  <xacro:property name="link_radius" value="0.01"/>
+  <xacro:property name="link1_length" value="0.15"/>
+  <xacro:property name="link2_length" value="0.5"/>
+  <xacro:property name="link3_length" value="0.5"/>
+  <xacro:property name="link4_length" value="0.15"/>
+  <xacro:property name="link5_length" value="0.10"/>
+  <xacro:property name="link6_length" value="0.05"/>
+  <!-- colors -->
+  <material name="joint_part1">
+    <color rgba="0.525 0.713 0.662 1.0"/>
+  </material>
+  <material name="joint_part2">
+    <color rgba="0.462 0.196 0.411 1.0"/>
+  </material>
+  <material name="base">
+    <color rgba="0.956863 0.796078 0.631373 1.0"/>
+  </material>
+  <material name="tip">
+    <color rgba="0.956 0.450 0.243 1.0"/>
+  </material>
+  <material name="link1">
+    <color rgba="0.949 0.631 0.823 1.0"/>
+  </material>
+  <material name="link2">
+    <color rgba="0.133 0.827 0.435 1.0"/>
+  </material>
+  <material name="link3">
+    <color rgba="0.968 0.721 0.313 1.0"/>
+  </material>
+  <material name="link4">
+    <color rgba="0.52549 0.529412 0.647059 1.0"/>
+  </material>
+  <material name="link5">
+    <color rgba="0.478431 0.415686 0.662745 1.0"/>
+  </material>
+  <material name="link6">
+    <color rgba="0.988 0.580 0.450 1.0"/>
+  </material>
+  <!-- Connect to world -->
+  <link name="world"/>
+  <joint name="world_joint" type="fixed">
+    <parent link="world"/>
+    <child link="base_link"/>
+    <origin xyz="0.0 0.0 0.0" rpy="0.0 0.0 0.0"/>
+  </joint>
+  <link name="base_link">
+    <inertial>
+      <origin xyz="0 0 ${joint_length / 2.0}" rpy="0 0 0"/>
+      <mass value="1"/>
+      <inertia ixx="1.0" ixy="0" ixz="0" iyy="1.0" iyz="0" izz="1.0"/>
+    </inertial>
+    <visual name="base">
+      <origin xyz="0 0 ${joint_length / 2.0}" rpy="0 0 0"/>
+      <geometry>
+        <cylinder length="${joint_length}" radius="${joint_radius}"/>
+      </geometry>
+      <material name="base"/>
+    </visual>
+  </link>
+  <joint name="joint1" type="revolute">
+    <parent link="base_link"/>
+    <child link="link1"/>
+    <origin xyz="0.0 0.0 ${3.0 / 2.0 * joint_length}" rpy="0.0 0.0 0.0"/>
+    <axis xyz="0 0 1"/>
+    <limit lower="${-2.0 * pi}" upper="${2.0 * pi}" effort="1.0" velocity="10.0"/>
+  </joint>
+  <link name="link1">
+    <inertial>
+      <origin xyz="0 0 ${link1_length / 2.0}" rpy="0 0 0"/>
+      <mass value="1"/>
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